Commit message: Ignore realsense pkg. Fix path to mesh.

File: realsense2_description/urdf/_d415.urdf.xacro (robot description, xacro)
@@ -46,5 +46,5 @@
           <origin xyz="${d415_cam_mount_from_center_offset} ${-d415_cam_depth_py} 0" rpy="${M_PI/2} 0 ${M_PI/2}"/>
           <geometry>
-            <mesh filename="package://realsense2_description/meshes/d415.stl" />
+            <mesh filename="file://$(find realsense2_description)/meshes/d415.stl" />
           </geometry>
           <material name="aluminum"/>
